Commit message: disable other collisions in urdf except torso thigh shank foot toe

File: engineai_legged_gym/resources/robots/prestoe/urdf/prestoe_less_noco.urdf (robot description, URDF)
Before this commit: robot d_biped, 25 links, 24 joints
Links:
- removed link L_elbowpitch_link
- removed link L_shoulderpitch_link
- removed link L_shoulderroll_link
- removed link L_shoulderyaw_link
- removed link R_elbowpitch_link
- removed link R_shoulderpitch_link
- removed link R_shoulderroll_link
- removed link R_shoulderyaw_link
- added link L_heel_contact
- added link L_toe_contact_1
- added link L_toe_contact_2
- added link L_toe_contact_3
- added link L_toe_contact_4
- added link R_heel_contact
- added link R_toe_contact_1
- added link R_toe_contact_2
- added link R_toe_contact_3
- added link R_toe_contact_4
- link L_ankle_link: geometry visual mesh filename=../meshes/ankle_pitch_link.dae
- link L_foot_link: geometry collision mesh filename=../meshes/foot_link.dae; visual mesh filename=../meshes/foot_link.dae
- link L_hippitch_link: geometry collision box size=0.08 0.08 0.28; visual mesh filename=../meshes/l_thigh_link.dae
- link L_hiproll_link: geometry visual mesh filename=../meshes/l_hip_roll_link.dae
- link L_hipyaw_link: geometry visual mesh filename=../meshes/hip_yaw_link.dae
- link L_shank_link: geometry collision box size=0.08 0.08 0.35; visual mesh filename=../meshes/shank_link.dae
- link L_toe_link: geometry collision mesh filename=../meshes/toe_link.dae; visual mesh filename=../meshes/toe_link.dae
- link R_ankle_link: geometry visual mesh filename=../meshes/ankle_pitch_link.dae
- link R_foot_link: geometry collision mesh filename=../meshes/foot_link.dae; visual mesh filename=../meshes/foot_link.dae
- link R_hippitch_link: geometry collision box size=0.08 0.08 0.28; visual mesh filename=../meshes/r_thigh_link.dae
- link R_hiproll_link: geometry visual mesh filename=../meshes/r_hip_roll_link.dae
- link R_hipyaw_link: geometry visual mesh filename=../meshes/hip_yaw_link.dae
- link R_shank_link: geometry collision box size=0.08 0.08 0.35; visual mesh filename=../meshes/shank_link.dae
- link R_toe_link: geometry collision mesh filename=../meshes/toe_link.dae; visual mesh filename=../meshes/toe_link.dae
- link pelvis: geometry visual mesh filename=../meshes/pelvis_link.dae
- link torso_link: geometry collision box size=0.2 0.2 0.3; visual mesh filename=../meshes/torso_link.dae
Joints:
- removed joint L_elbowpitch
- removed joint L_hipyaw
- removed joint L_shoulderpitch
- removed joint L_shoulderroll
- removed joint L_shoulderyaw
- removed joint R_elbowpitch
- removed joint R_hipyaw
- removed joint R_shoulderpitch
- removed joint R_shoulderroll
- removed joint R_shoulderyaw
- removed joint fixed
- removed joint torsoyaw
- added joint L_heel_contact_joint: type fixed, parent L_foot_link, child L_heel_contact, origin xyz=-63.374e-3 0 -51.76e-3 rpy=0 0 0
- added joint L_toe_contact_joint_1: type fixed, parent L_toe_link, child L_toe_contact_1, origin xyz=69e-3 30e-3 -44.9e-3 rpy=0 0 0
- added joint L_toe_contact_joint_2: type fixed, parent L_toe_link, child L_toe_contact_2, origin xyz=-4e-3 33e-3 -44.9e-3 rpy=0 0 0
- added joint L_toe_contact_joint_3: type fixed, parent L_toe_link, child L_toe_contact_3, origin xyz=69e-3 -30e-3 -44.9e-3 rpy=0 0 0
- added joint L_toe_contact_joint_4: type fixed, parent L_toe_link, child L_toe_contact_4, origin xyz=-4e-3 -33e-3 -44.9e-3 rpy=0 0 0
- added joint R_heel_contact_joint: type fixed, parent R_foot_link, child R_heel_contact, origin xyz=-64.374e-3 0 -51.76e-3 rpy=0 0 0
- added joint R_toe_contact_joint_1: type fixed, parent R_toe_link, child R_toe_contact_1, origin xyz=69e-3 30e-3 -44.9e-3 rpy=0 0 0
- added joint R_toe_contact_joint_2: type fixed, parent R_toe_link, child R_toe_contact_2, origin xyz=-4e-3 33e-3 -44.9e-3 rpy=0 0 0
- added joint R_toe_contact_joint_3: type fixed, parent R_toe_link, child R_toe_contact_3, origin xyz=69e-3 -30e-3 -44.9e-3 rpy=0 0 0
- added joint R_toe_contact_joint_4: type fixed, parent R_toe_link, child R_toe_contact_4, origin xyz=-4e-3 -33e-3 -44.9e-3 rpy=0 0 0
- added joint a_torsoyaw: type fixed, parent torso_link, child pelvis, origin xyz=0.0 0.0 -44.5e-3 rpy=0 0 0, axis 0 0 1, limit lower=-1.57079632679 upper=1.57079632679 effort=1000 velocity=20
- added joint bR_hipyaw: type revolute, parent pelvis, child R_hipyaw_link, origin xyz=0 -54.71371e-3 -48.37244e-3 rpy=-0.2618 0 0, axis 0 0 1, limit lower=-1.57 upper=1.57 effort=100.0 velocity=20.0
- added joint cL_hipyaw: type revolute, parent pelvis, child L_hipyaw_link, origin xyz=0 54.71371e-3 -48.37244e-3 rpy=0.2618 0 0, axis 0 0 1, limit lower=-1.570796 upper=1.570796 effort=100 velocity=20
- added joint floating_base_joint: type floating, parent world, child torso_link
- joint R_anklepitch: limit lower=-1.57 upper=1.57 effort=0.0 velocity=20.0 -> lower=-1.57 upper=1.57 effort=100.0 velocity=20.0
- joint R_ankleroll: limit lower=-0.785 upper=0.785 effort=0.0 velocity=20.0 -> lower=-0.785 upper=0.785 effort=100.0 velocity=20.0
- joint R_hiproll: limit lower=-1.57 upper=1.57 effort=0.0 velocity=20.0 -> lower=-1.57 upper=1.57 effort=100.0 velocity=20.0
- joint R_knee: limit lower=0.0 upper=2.61799 effort=0.0 velocity=20.0 -> lower=0.0 upper=2.61799 effort=100.0 velocity=20.0
- joint R_toepitch: limit lower=-0.5236 upper=0.5236 effort=0.0 velocity=20.0 -> lower=-0.5236 upper=0.5236 effort=100.0 velocity=20.0
